Commit message: Working UDRF launch

File: test_bench_ws/src/test_bench/urdf/FLIR.xacro (robot description, xacro)
@@ -16,5 +16,5 @@
     </link>
     <joint name="FLIR_joint" type="fixed">
-        <parent link="bench_joint"/>
+        <parent link="bench_footprint"/>
         <child link="FLIR"/>
         <origin xyz="${FLIR_xyz}" rpy="${FLIR_rot}"/>

File: test_bench_ws/src/test_bench/urdf/LIDAR.xacro (robot description, xacro)
@@ -16,5 +16,5 @@
     </link>
     <joint name="LIDAR_joint" type="fixed">
-        <parent link="bench_joint"/>
+        <parent link="bench_footprint"/>
         <child link="LIDAR"/>
         <origin xyz="${LIDAR_xyz}" rpy="${LIDAR_rot}"/>
