Commit message: updated urdg

File: test_bench_ws/src/test_bench/urdf/REALSENSE.xacro (robot description, xacro)
@@ -21,5 +21,5 @@
     </joint>
     <!-- RS Camera Link-->
-    <link name="camera" type="fixed">
+    <link name="camera_link" type="fixed">
     </link>
     <joint name="camera_joint" type="fixed">
