Commit message: modified

File: ROS2_Master/test_bench_ws/src/test_bench/urdf/FLIR.xacro (robot description, xacro)
@@ -16,5 +16,5 @@
     </link>
     <joint name="FLIR_joint" type="fixed">
-        <parent link="bench_footprint"/>
+        <parent link="zero_point"/>
         <child link="FLIR"/>
         <origin xyz="${FLIR_xyz}" rpy="${FLIR_rot}"/>

File: ROS2_Master/test_bench_ws/src/test_bench/urdf/LIDAR.xacro (robot description, xacro)
@@ -16,5 +16,5 @@
     </link>
     <joint name="LIDAR_joint" type="fixed">
-        <parent link="bench_footprint"/>
+        <parent link="zero_point"/>
         <child link="LIDAR"/>
         <origin xyz="${LIDAR_xyz}" rpy="${LIDAR_rot}"/>

File: ROS2_Master/test_bench_ws/src/test_bench/urdf/REALSENSE.xacro (robot description, xacro)
@@ -16,5 +16,5 @@
     </link>
     <joint name="RS_joint" type="fixed">
-        <parent link="bench_footprint"/>
+        <parent link="zero_point"/>
         <child link="RS"/>
         <origin xyz="${RS_xyz}" rpy="${RS_rot}"/>

File: ROS2_Master/test_bench_ws/src/test_bench/urdf/test_bench_core.xacro (robot description, xacro)
@@ -1,11 +1,12 @@
 <?xml version="1.0"?>
 <robot xmlns:xacro="http://www.ros.org/wiki/xacro">
-    <!-- Test Bench Properties-->
-    <xacro:property name="bench_width" value="1.2"/>
-    <xacro:property name="bench_length" value=".6"/>
-    <xacro:property name="bench_height" value=".5"/>
-    <xacro:property name="wheel_radius" value="0.10"/>
-    <xacro:property name="wheel_width" value="0.04"/>
-    <xacro:property name="wheel_offset" value=".1"/>
+    <!-- Test Bench Properties, Values in Meters-->
+    <xacro:property name="bench_width" value="1.198"/>
+    <xacro:property name="bench_depth" value=".7"/>
+    <xacro:property name="bench_base_height" value=".804"/>
+    <xacro:property name="bench_wall_height" value=".808"/>
+    <xacro:property name="bench_wall_depth" value=".063"/>
+    <xacro:property name="wheel_radius" value="0.0625"/>
+    <xacro:property name="wheel_offset" value=".031"/>
     <!-- Base Link, this is our origin point for all test bench joints-->
     <link name="base_link">
@@ -15,5 +16,5 @@
         <visual>
             <geometry>
-                <box size="${bench_length} ${bench_width} ${bench_height}"/>
+                <box size="${bench_length} ${(bench_depth + bench_wall_depth)} ${(bench_base_height+bench_wall_height)}"/>
             </geometry>
             <material name="Cyan">
@@ -27,3 +28,10 @@
         <origin xyz="0.0 0.0 ${(wheel_radius*2+wheel_offset)}" rpy="0 0 0"/>
     </joint>
+    <link name="zero_point" type="fixed">
+    </link>
+        <joint name="zero_joint" type="fixed">
+        <parent link="bench_footprint"/>
+        <child link="zero_point"/>
+        <origin xyz="{(-bench_width/2)} {(-(bench_depth + bench_wall_depth)/2)} ${bench_base_height}" rpy="0 0 0"/>
+    </joint>
 </robot>
