Commit message: urdf and marvelmind

File: ROS2_Master/test_bench_ws/src/test_bench/urdf/test_bench.urdf.xacro (robot description, xacro)
@@ -5,3 +5,5 @@
     <xacro:include filename="LIDAR.xacro"/>
     <xacro:include filename="REALSENSE.xacro"/>
+    <xacro:include filename="MARVELMIND.xacro"/>
+    <xacro:include filename="BNO055.xacro"/>
 </robot>

File: ROS2_Master/test_bench_ws/src/test_bench/urdf/test_bench_core.xacro (robot description, xacro)
@@ -16,8 +16,18 @@
         <visual>
             <geometry>
-                <box size="${bench_length} ${(bench_depth + bench_wall_depth)} ${(bench_base_height+bench_wall_height)}"/>
+                <box size="${bench_width} ${(bench_depth + bench_wall_depth)} ${(bench_base_height+bench_wall_height)}"/>
             </geometry>
-            <material name="Cyan">
-                <color rgba="0 1.0 1.0 1.0"/>
+            <material name="Grey">
+                <color rgba=".1 .1 .1 .1"/>
+            </material>
+        </visual>
+    </link>
+    <link name="bench_wall" type="fixed">
+        <visual>
+            <geometry>
+                <box size="${bench_width} ${bench_wall_depth} ${bench_wall_height}"/>
+            </geometry>
+            <material name="Grey">
+                <color rgba=".1 .1 .1 .1"/>
             </material>
         </visual>
@@ -28,4 +38,9 @@
         <origin xyz="0.0 0.0 ${(wheel_radius*2+wheel_offset)}" rpy="0 0 0"/>
     </joint>
+    <joint name="wall_joint" type="fixed">
+        <parent link="bench_footprint"/>
+        <child link="bench_wall"/>
+        <origin xyz="0.0 ${(bench_depth+(bench_wall_depth/2))} ${bench_base_height}" rpy="0 0 0"/>
+    </joint>
     <link name="zero_point" type="fixed">
     </link>
@@ -33,5 +48,5 @@
         <parent link="bench_footprint"/>
         <child link="zero_point"/>
-        <origin xyz="{(-bench_width/2)} {(-(bench_depth + bench_wall_depth)/2)} ${bench_base_height}" rpy="0 0 0"/>
+        <origin xyz="${(-bench_width/2)} ${(-(bench_depth + bench_wall_depth)/2)} ${bench_base_height}" rpy="0 0 0"/>
     </joint>
 </robot>
