Commit message: Final commit from me.  Good luck.

File: ROS2_Master/test_bench_ws/src/test_bench/urdf/BNO055.xacro (robot description, xacro)
@@ -2,5 +2,5 @@
 <robot xmlns:xacro="http://www.ros.org/wiki/xacro">
     <xacro:property name="BNO_dims" value="0.1 0.1 0.1"/>
-    <xacro:property name="BNO_xyz" value="0.0 0.0 2.0"/>
+    <xacro:property name="BNO_xyz" value="0.587 0.68 .232"/>
     <xacro:property name="BNO_rot" value="0.0 0.0 0.0"/>
     <!-- BNO Link-->

File: ROS2_Master/test_bench_ws/src/test_bench/urdf/FLIR.xacro (robot description, xacro)
@@ -2,5 +2,5 @@
 <robot xmlns:xacro="http://www.ros.org/wiki/xacro">
     <xacro:property name="FLIR_dims" value="0.1 0.1 0.1"/>
-    <xacro:property name="FLIR_xyz" value="0.0 0.0 2.0"/>
+    <xacro:property name="FLIR_xyz" value=".938 0.63 .34"/>
     <xacro:property name="FLIR_rot" value="0.0 0.0 0.0"/>
     <!-- FLIR Link-->

File: ROS2_Master/test_bench_ws/src/test_bench/urdf/LIDAR.xacro (robot description, xacro)
@@ -2,5 +2,5 @@
 <robot xmlns:xacro="http://www.ros.org/wiki/xacro">
     <xacro:property name="LIDAR_dims" value="0.1 0.1 0.1"/>
-    <xacro:property name="LIDAR_xyz" value="0.0 0.0 2.0"/>
+    <xacro:property name="LIDAR_xyz" value="0.26 0.495 0.69"/>
     <xacro:property name="LIDAR_rot" value="0.0 0.0 0.0"/>
     <!-- LIDAR Link-->

File: ROS2_Master/test_bench_ws/src/test_bench/urdf/MARVELMIND.xacro (robot description, xacro)
@@ -2,5 +2,5 @@
 <robot xmlns:xacro="http://www.ros.org/wiki/xacro">
     <xacro:property name="MM_dims" value="0.1 0.1 0.1"/>
-    <xacro:property name="MM_xyz" value="0.0 0.0 2.0"/>
+    <xacro:property name="MM_xyz" value="1.18 .72 .808"/>
     <xacro:property name="MM_rot" value="0.0 0.0 0.0"/>
     <!-- MM Link-->

File: ROS2_Master/test_bench_ws/src/test_bench/urdf/REALSENSE.xacro (robot description, xacro)
@@ -2,5 +2,5 @@
 <robot xmlns:xacro="http://www.ros.org/wiki/xacro">
     <xacro:property name="RS_dims" value="0.1 0.1 0.1"/>
-    <xacro:property name="RS_xyz" value="0.0 0.0 2.0"/>
+    <xacro:property name="RS_xyz" value=".780 .68 .615"/>
     <xacro:property name="RS_rot" value="0.0 0.0 0.0"/>
     <!-- RS Link-->

File: ROS2_Master/test_bench_ws/src/test_bench/urdf/test_bench.urdf.xacro (robot description, xacro)
@@ -7,3 +7,4 @@
     <xacro:include filename="MARVELMIND.xacro"/>
     <xacro:include filename="BNO055.xacro"/>
+    <xacro:include filename="GPS.xacro"/>
 </robot>
